File: feeder/pcb/mobo/mobo.kicad_pcb (KiCad board)
At the start: 2 copper layers, 200 x 100 mm, 88 parts, among them J1 SWD_10, J2 FTDI_HEADER, J3 PLATED_PADS, M1 PEEL_MOTOR, M2 DRIVE_MOTOR, SW1 RESET, SW2 BUTTON_1, SW3 BUTTON_2, SW4 BOOT, U1 QRE1113GR, U2 STM32F103C8Tx, U3 TCS40DPR, U4 AP1117-33, U5 MCP16301, U6 DRV8833PWP, U7 MAX3078E, Y1 8MHz

Commit message: reworked feeder pcb to have minimal dimensions, more available parts, and swappable uC options
Parts:
- removed C15: 100n, Capacitor_SMD:C_0805_2012Metric
- removed D7: 1N4148, Diode_SMD:D_SOD-123
- removed the G*** at (178.3, 58.8)
- removed the G*** at (195.9, 58.8)
- removed J2: FTDI_HEADER, Connector_PinHeader_2.54mm:PinHeader_1x06_P2.54mm_Vertical
- removed M1: PEEL_MOTOR, Connector_PinHeader_2.54mm:PinHeader_1x02_P2.54mm_Vertical
- removed M2: DRIVE_MOTOR, Connector_PinHeader_2.54mm:PinHeader_1x02_P2.54mm_Vertical
- removed R12, R4: 10k, Resistor_SMD:R_0805_2012Metric
- removed SW4: BOOT, Button_Switch_SMD:Panasonic_EVQPUJ_EVQPUA
- removed svg2mod (x26): G***, label
- added G***: LOGO, index:goblin, F.Cu at (-4.60, -36.8)
- added J4: PEEL_MOTOR, Connector_PinHeader_2.54mm:PinHeader_1x06_P2.54mm_Vertical, F.Cu at (-17.8, 10.2)
- added J5: Conn_01x07_Female, index:AVX-9155-005-541, F.Cu at (-4.25, 7.75)
- added U8: DRV8837, Package_SON:WSON-8-1EP_2x2mm_P0.5mm_EP0.9x1.6mm, F.Cu at (-33.5, 17.0)
- C10: value 100n -> 4.7uF
- C11, C8: value 4.7u -> 4.7uF
- C12: value 10n -> 100uF; footprint Capacitor_SMD:C_0805_2012Metric -> Capacitor_SMD:C_Elec_5x5.8
- C14: value 1uF -> 470pF
- C16: value 10u -> 470uF; footprint Capacitor_SMD:C_0805_2012Metric -> Capacitor_SMD:C_Elec_5x5.8
- C17: value 10n -> 100n
- C18, C20: value 10u -> 100n
- C19: value 2.2u -> 100n
- C7: value 4.7u -> 100n
- D6: value B140 -> 1N5819; footprint Diode_SMD:D_SMB_Handsoldering -> Diode_SMD:D_SOD-123
- J3: value PLATED_PADS -> DRIVE_MOTOR; footprint index:5-pad-spring-finger-interface -> Connector_PinHeader_2.54mm:PinHeader_1x06_P2.54mm_Vertical
- L1: value 15u -> 220uH; footprint Inductor_SMD:L_Taiyo-Yuden_NR-50xx_HandSoldering -> Inductor_SMD:L_6.3x6.3_H3
- R1: value 100 -> 1k
- R10: value 1k -> 10k
- R11: value 56k -> 10k
- R6: value 10k -> 1.2k
- R9: value 10k -> 3.6k
- U1: value QRE1113GR -> STM32F031C6Tx; footprint OptoDevice:OnSemi_CASE100CY -> Package_QFP:LQFP-48_7x7mm_P0.5mm
- U2: value STM32F103C8Tx -> STM32F031K6Ux; footprint Package_QFP:LQFP-48_7x7mm_P0.5mm -> Package_DFN_QFN:QFN-32-1EP_5x5mm_P0.5mm_EP3.45x3.45mm
- U5: value MCP16301 -> MC34063AD; footprint Package_TO_SOT_SMD:SOT-23-6 -> Package_SO:SOIC-8_3.9x4.9mm_P1.27mm
- U6: value DRV8833PWP -> MAX3078E; footprint Package_SO:HTSSOP-16-1EP_4.4x5mm_P0.65mm_EP3.4x5mm_Mask2.46x2.31mm_ThermalVias -> Package_SO:SOIC-8_3.9x4.9mm_P1.27mm
- U7: value MAX3078E -> DRV8837; footprint Package_SO:SOIC-8_3.9x4.9mm_P1.27mm -> Package_SON:WSON-8-1EP_2x2mm_P0.5mm_EP0.9x1.6mm
- moved FID3 230.6 mm to (-2.80, -44.5), turned to 0 degrees
- moved J3 164.7 mm to (-17.8, 12.7), turned to -90 degrees
- moved U7 160.3 mm to (-26.1, 17.0), turned to -90 degrees
- moved R11 160.3 mm to (-31.6, 20.0), turned to 0 degrees
- moved C7 159.4 mm to (-35.9, 24.1), turned to 0 degrees
- moved C11 152.5 mm to (-32.2, 27.3)
- moved SW1 143.0 mm to (-36.0, 38.0)
- moved C18 141.7 mm to (-28.6, 17.0), turned to -90 degrees
- moved FID1 136.7 mm to (-34.2, 8.70), turned to 0 degrees
- moved U5 134.8 mm to (-10.1, 19.9), turned to 90 degrees
- moved C9 134.4 mm to (-9.80, 30.0), turned to 180 degrees
- moved C13 130.3 mm to (-13.0, 31.1), turned to 90 degrees
- moved U4 125.7 mm to (-4.70, 36.1)
- moved L1 125.1 mm to (-3.70, 22.1)
- moved R1 125.1 mm to (-32.2, 33.6), turned to -90 degrees
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Connections:
- C1 pad 1: Net-(C1-Pad1) -> OSC_IN
- C10 pad 2: BOOT0 -> +3V3
- C11 pad 1: +VDC -> GND
- C11 pad 2: GND -> +3V3
- C12 pad 1: +3V3 -> +VDC
- C14 pad 1: +3V3 -> GND
- C14 pad 2: GND -> Net-(C14-Pad2)
- C17 pad 1: +5V -> GND
- C17 pad 2: Net-(C17-Pad2) -> +5V
- C18 pad 1: +5V -> GND
- C18 pad 2: GND -> +3V3
- C19 pad 1: Net-(C19-Pad1) -> GND
- C19 pad 2: GND -> +5V
- C2 pad 1: Net-(C2-Pad1) -> OSC_OUT
- C20 pad 1: +5V -> GND
- C20 pad 2: GND -> +3V3
- C3 pad 2: RESET -> +3V3
- C4 pad 1: +3V3 -> GND
- C4 pad 2: GND -> +3V3
- C5 pad 1: +3V3 -> GND
- C5 pad 2: GND -> +3V3
- C6 pad 1: +3V3 -> GND
- C6 pad 2: GND -> RESET
- C7 pad 1: +VDC -> GND
- C7 pad 2: GND -> +3V3
- C8 pad 1: +3V3 -> GND
- C8 pad 2: GND -> +3V3
- D6 pad 1: Net-(C15-Pad2) -> Net-(D6-Pad1)
- J1 pad 6: Net-(J1-Pad6) -> unconnected-(J1-Pad6)
- J1 pad 7: Net-(J1-Pad7) -> unconnected-(J1-Pad7)
- J1 pad 8: Net-(J1-Pad8) -> unconnected-(J1-Pad8)
- J3 pad 1: +VDC -> +3V3
- J3 pad 2: RS-485+ -> GND
- J3 pad 3: RS-485- -> DRIVE_QUAD_A
- J3 pad 4: 1WIRE -> DRIVE_QUAD_B
- J3 pad 5: GND -> DRIVE_M1
- L1 pad 1: Net-(C15-Pad2) -> Net-(D6-Pad1)
- R1 pad 1: +3V3 -> 1WIRE
- R1 pad 2: Net-(R1-Pad2) -> +3V3
- R10 pad 1: 1WIRE -> Net-(R10-Pad1)
- R11 pad 1: +5V -> Net-(R11-Pad1)
- R11 pad 2: Net-(R11-Pad2) -> +3V3
- R6 pad 1: GND -> Net-(R6-Pad1)
- R6 pad 2: Net-(R6-Pad2) -> GND
- R9 pad 1: GND -> Net-(R6-Pad1)
- R9 pad 2: Net-(R9-Pad2) -> +5V
- U1 pad 1: Net-(R1-Pad2) -> +3V3
- U1 pad 2: GND -> unconnected-(U1-Pad2)
- U1 pad 3: OPTO_SIG_QRE1113 -> unconnected-(U1-Pad3)
- U1 pad 4: GND -> unconnected-(U1-Pad4)
- U2 pad 10: Net-(U2-Pad10) -> DRIVE_QUAD_A
- U2 pad 11: OPTO_SIG_VCNT2020 -> unconnected-(U2-Pad11)
- U2 pad 12: 1WIRE -> PEEL_QUAD_A
- U2 pad 13: FILM_TENSION -> PEEL_QUAD_B
- U2 pad 14: OPTO_SIG_QRE1113 -> unconnected-(U2-Pad14)
- U2 pad 15: SW1 -> LED2
- U2 pad 16: SW2 -> LED3
- U2 pad 17: LED2 -> +3V3
- U2 pad 19: LED5 -> MCU_TX
- U2 pad 2: Net-(U2-Pad2) -> OSC_IN
- U2 pad 20: Net-(R6-Pad2) -> MCU_RX
- U2 pad 21: LED4 -> ~{RE}
- U2 pad 22: LED3 -> DE
- U2 pad 23: GND -> SWDIO
- U2 pad 24: +3V3 -> SWCLK
- U2 pad 25: Net-(U2-Pad25) -> DRIVE_QUAD_B
- U2 pad 26: Net-(U2-Pad26) -> LED4
- U2 pad 27: Net-(U2-Pad27) -> LED5
- U2 pad 28: Net-(U2-Pad28) -> DRIVE1
- U2 pad 29: Net-(U2-Pad29) -> DRIVE2
- U2 pad 3: Net-(U2-Pad3) -> OSC_OUT
- U2 pad 30: MCU_TX -> PEEL1
- U2 pad 31: MCU_RX -> BOOT0
- U2 pad 32: ~{RE} -> PEEL2
- U2 pad 33: DE -> GND
- U2 pad 4: Net-(U2-Pad4) -> RESET
- U2 pad 5: Net-(C1-Pad1) -> +3V3
- U2 pad 6: Net-(C2-Pad1) -> 1WIRE
- U2 pad 7: RESET -> FILM_TENSION
- U2 pad 8: GND -> SW1
- U2 pad 9: +3V3 -> SW2
- U5 pad 1: Net-(C15-Pad1) -> Net-(U5-Pad1)
- U5 pad 2: GND -> Net-(D6-Pad1)
- U5 pad 3: Net-(R11-Pad2) -> Net-(C14-Pad2)
- U5 pad 4: +VDC -> GND
- U5 pad 5: +VDC -> Net-(R6-Pad1)
- U5 pad 6: Net-(C15-Pad2) -> +VDC
- U6 pad 1: +5V -> MCU_RX
- U6 pad 2: Net-(M2-Pad1) -> ~{RE}
- U6 pad 3: GND -> DE
- U6 pad 4: Net-(M2-Pad2) -> MCU_TX
- U6 pad 5: Net-(M1-Pad1) -> GND
- U6 pad 6: GND -> RS-485+
- U6 pad 7: Net-(M1-Pad2) -> RS-485-
- U6 pad 8: Net-(U6-Pad8) -> +3V3
- U7 pad 1: MCU_RX -> +5V
- U7 pad 2: ~{RE} -> DRIVE_M1
- U7 pad 3: DE -> DRIVE_M2
- U7 pad 4: MCU_TX -> GND
- U7 pad 5: GND -> DRIVE2
- U7 pad 6: RS-485+ -> DRIVE1
- U7 pad 7: RS-485- -> Net-(R10-Pad1)
- Y1 pad 1: Net-(C1-Pad1) -> OSC_IN
- Y1 pad 3: Net-(C2-Pad1) -> OSC_OUT
Routing:
- net +3V3: track 396.4 -> 218.6 mm, vias 8 -> 10
- net RS-485-: track 100.8 -> 3.66 mm, vias 2 -> 0
- net RS-485+: track 100.7 -> 3.70 mm, vias 2 -> 0
- net +VDC: track 91.6 -> 9.02 mm
- net 1WIRE: track 142.3 -> 60.8 mm
- net FILM_TENSION: track 99.2 -> 32.9 mm
- net Net-(M1-Pad1): track 55.3 -> 0.00 mm
- net Net-(M2-Pad2): track 52.5 -> 0.00 mm, vias 2 -> 0
- net OPTO_SIG_QRE1113: track 48.8 -> 0.00 mm, vias 2 -> 0
- net Net-(M1-Pad2): track 47.5 -> 0.00 mm
- net Net-(M2-Pad1): track 45.7 -> 0.00 mm, vias 2 -> 0
- net PEEL_QUAD_A: track 0.00 -> 42.4 mm, vias 0 -> 1
- net PEEL_QUAD_B: track 0.00 -> 40.5 mm, vias 0 -> 1
- net DRIVE_QUAD_A: track 0.00 -> 39.0 mm, vias 0 -> 1
- net Net-(R9-Pad2): track 35.6 -> 0.00 mm, vias 2 -> 0
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Other:
- board size 200 x 100 mm -> 40 x 88 mm
- board text added: "Feeder Mobo REV06-BETA0 Opulo Inc."
- board text removed: "<<hash>>"
