File: pnp/pcb/mobo/aux_header.kicad_sch (KiCad schematic)
At the start: 1 part, among them J20 AUX

Commit message: another huge chunk of work on rev04 of the mobo. breaks out diag and index pin for TMC2209 sensorless homing. reduces unique part count by consolidating resistor values where possible. replaces full ADC pipeline with monolithic I2C vacuum sensor and an I2C multiplexer due to address collision issues with two sensors. adds solder selectable jumpers for selecting whether an axis uses switch or TMC homing. redoes lots of routing of the SPI lines up to the stepper drivers.
Other:
- company: (none) -> Opulo
- title: (none) -> LumenPnP Motherboard
Changed lines of the file:
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@@
   (paper "A4")
   (title_block
+    (title "LumenPnP Motherboard")
     (date "2022-03-29")
+    (company "Opulo")
   )
   (hierarchical_label "PWM1" (shape bidirectional) (at 138.43 97.155 180)
@@
   (symbol (lib_id "power:GND") (at 151.13 92.075 90)
     (in_bom yes) (on_board yes)
-    (property "Reference" "#PWR0235" (id 0) (at 157.48 92.075 0)
+    (property "Reference" "#PWR0238" (id 0) (at 157.48 92.075 0)
       (effects (font (size 1.27 1.27)) hide)
     )
@@
   (symbol (lib_id "power:VDC") (at 138.43 92.075 90)
     (in_bom yes) (on_board yes)
-    (property "Reference" "#PWR0233" (id 0) (at 140.97 92.075 0)
+    (property "Reference" "#PWR0236" (id 0) (at 140.97 92.075 0)
       (effects (font (size 1.27 1.27)) hide)
     )
@@
   (symbol (lib_id "power:+3.3V") (at 138.43 94.615 90)
     (in_bom yes) (on_board yes)
-    (property "Reference" "#PWR0234" (id 0) (at 142.24 94.615 0)
+    (property "Reference" "#PWR0237" (id 0) (at 142.24 94.615 0)
       (effects (font (size 1.27 1.27)) hide)
     )
