File: pnp/pcb/mobo/aux_headers.kicad_sch (KiCad schematic)
At the start: 0 parts

Commit message: another huge chunk of work on rev04 of the mobo. breaks out diag and index pin for TMC2209 sensorless homing. reduces unique part count by consolidating resistor values where possible. replaces full ADC pipeline with monolithic I2C vacuum sensor and an I2C multiplexer due to address collision issues with two sensors. adds solder selectable jumpers for selecting whether an axis uses switch or TMC homing. redoes lots of routing of the SPI lines up to the stepper drivers.
Other:
- company: (none) -> Opulo
- title: Output -> LumenPnP Motherboard
Changed lines of the file:
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@@
   (paper "A4")
   (title_block
-    (title "Output")
+    (title "LumenPnP Motherboard")
     (date "2022-03-29")
     (rev "003")
+    (company "Opulo")
   )
   (junction (at 85.09 73.66) (diameter 0) (color 0 0 0 0)
