File: pnp/pcb/mobo/servos.kicad_sch (KiCad schematic)
At the start: 2 parts, among them J15 SERVO1, J16 SERVO2

Commit message: another huge chunk of work on rev04 of the mobo. breaks out diag and index pin for TMC2209 sensorless homing. reduces unique part count by consolidating resistor values where possible. replaces full ADC pipeline with monolithic I2C vacuum sensor and an I2C multiplexer due to address collision issues with two sensors. adds solder selectable jumpers for selecting whether an axis uses switch or TMC homing. redoes lots of routing of the SPI lines up to the stepper drivers.
Other:
- company: (none) -> Opulo
- title: (none) -> LumenPnP Motherboard
Changed lines of the file:
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@@
   (paper "A4")
   (title_block
+    (title "LumenPnP Motherboard")
     (date "2022-03-29")
+    (company "Opulo")
   )
   (wire (pts (xy 148.59 106.68) (xy 149.86 106.68))
