File: pnp/pcb/mobo/motor_control.kicad_sch (KiCad schematic)
At the start: 0 parts

Commit message: fixes erc errors about pin connectivity
Other:
- sheet Motor AUX ports: added none; removed INDEX
- sheet Motor X ports: added none; removed INDEX
- sheet Motor Y ports: added none; removed INDEX
- sheet Motor Z ports: added none; removed INDEX
- sheet Motor left ports: added none; removed INDEX
- sheet Motor right ports: added none; removed INDEX
Changed lines of the file:
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@@
-      (effects (font (size 1.27 1.27)) (justify left))
-    )
-    (pin "INDEX" input (at 36.83 118.11 180)
       (effects (font (size 1.27 1.27)) (justify left))
     )
@@
     )
     (pin "CIPO" output (at 204.47 97.79 180)
-      (effects (font (size 1.27 1.27)) (justify left))
-    )
-    (pin "INDEX" input (at 204.47 118.11 180)
       (effects (font (size 1.27 1.27)) (justify left))
     )
@@
       (effects (font (size 1.27 1.27)) (justify left))
     )
-    (pin "INDEX" input (at 78.74 118.11 180)
-      (effects (font (size 1.27 1.27)) (justify left))
-    )
   )
   (sheet (at 162.56 90.17) (size 27.94 30.48)
@@
     )
     (pin "CS_UART" input (at 162.56 100.33 180)
-      (effects (font (size 1.27 1.27)) (justify left))
-    )
-    (pin "INDEX" input (at 162.56 118.11 180)
       (effects (font (size 1.27 1.27)) (justify left))
     )
@@
       (effects (font (size 1.27 1.27)) (justify left))
     )
-    (pin "INDEX" input (at 246.38 118.11 180)
-      (effects (font (size 1.27 1.27)) (justify left))
-    )
     (pin "DIAG" input (at 246.38 115.57 180)
       (effects (font (size 1.27 1.27)) (justify left))
@@
       (effects (font (size 1.27 1.27)) (justify left))
     )
-    (pin "INDEX" input (at 120.65 118.11 180)
-      (effects (font (size 1.27 1.27)) (justify left))
-    )
